File: RESTORE_AVR_FUSES_SMD.kicad_pcb (KiCad board)
At the start: 2 copper layers, 68.6 x 53.3 mm, 45 parts, among them Q1 MMBT2222A, Q2 MMBT2222A, Q3 MMBT2222A, SW1 START, SW2 RESET, U1 MCP23S08

Commit message: 25/03/23/A
Parts:
- removed G***: LOGO, x_Logos:xdna_electronics_design_round_skill

Commit message: 26/12/13/A
Parts:
- added G***: LOGO, x_Logos:xdna_electronics_design_round_skill, B.Cu at (107.6, 103.0)
